File: hardware/rev-a/carrier.kicad_pcb (KiCad board)
At the start: 2 copper layers, 68 x 70 mm, 24 parts, among them J1 LILYGO P1 / upper row, J2 LILYGO P2 / lower row, J3 MQ3 cable / 5V GND AO

Commit message: Resize carrier and case around measured MQ-3 sensor
Parts:
- moved TP8 37.7 mm to (150.0, 130.0)
- moved TP7 37.3 mm to (150.0, 125.0)
- moved J3 25.5 mm to (136.0, 128.0)
- moved S1 24.4 mm to (114.0, 122.0)
- moved R4 23.1 mm to (128.0, 129.0)
- moved H2 16.0 mm to (103.0, 131.0)
- moved H3 16.0 mm to (165.0, 131.0)
- moved TP6 12.1 mm to (162.0, 125.0)
- moved JP1 4.12 mm to (103.0, 111.0)
- moved TP5 4.12 mm to (156.0, 125.0)
Routing:
- net /+5V_SENSOR: track 89.6 -> 101.6 mm
- net /MQ3_AO: track 118.9 -> 128.6 mm
- net /ADC_GPIO1: track 85.2 -> 81.4 mm
- net /+5V_USB: track 23.5 -> 26.5 mm
- net /GND: track 12.2 -> 12.7 mm
Other:
- board size 68 x 70 mm -> 68 x 54 mm
- board text added: "68 x 54 mm / 1.6 mm / 2 layers"
- board text added: "ON"
- board text removed: "68 x 70 mm / 1.6 mm / 2 layers"
- board text removed: "FIT SHUNT"
